Commit message: Collision frame substituted in the robot description. Changed from the mesh to a box

File: iiwa_gripper_description/urdf/iiwa_gripper.urdf.xacro (robot description, xacro)
@@ -26,8 +26,8 @@
     </visual>
     <collision>
-      <origin xyz="0.4 0 0" rpy="-1.57 0 0"/>
+      <origin xyz="0.37 0 0.499" rpy="-1.57 0 0"/>
       <geometry>
-        <!--box size="0.77 1.0 0.6"/-->
-	      <mesh filename="package://iiwa_gripper_description/meshes/collision/suporte.stl"/>
+        <box size="0.77 1.0 0.6"/>
+	      <!--mesh filename="package://iiwa_gripper_description/meshes/collision/suporte.stl"/-->
       </geometry>
     </collision>

Commit message: Added a iiwa_surgery_description. The iiwa is on top of a support and has no tool attached

File: iiwa_gripper_description/urdf/iiwa_gripper.urdf.xacro (robot description, xacro)
@@ -18,15 +18,20 @@
   <!--     <link name="world"/> -->
   <link name="world">
+    <inertial>
+      <origin xyz="0.385 0.5 0.3" rpy="0 0 0"/>
+      <mass value="100"/>
+      <inertia ixx="11.33"  ixy="0"  ixz="0" iyy="13.27" iyz="0" izz="7.94" />
+    </inertial>
     <visual>
       <origin xyz="0.4 0 0" rpy="-1.57 0 0"/>
       <geometry>
         <!--box size="0.77 1.0 0.6"/-->
-	      <mesh filename="package://iiwa_gripper_description/meshes/collision/suporte.stl"/>
+	      <mesh filename="package://iiwa_surgery_description/meshes/collision/suporte.stl"/>
       </geometry>
     </visual>
     <collision>
-      <origin xyz="0.37 0 0.499" rpy="-1.57 0 0"/>
+      <origin xyz="0.40 0 0.499" rpy="-1.57 0 0"/>
       <geometry>
-        <box size="0.77 1.0 0.6"/>
+        <box size="0.75 1.0 0.6"/>
 	      <!--mesh filename="package://iiwa_gripper_description/meshes/collision/suporte.stl"/-->
       </geometry>

Commit message: Moveit can be initialized from the python script

File: iiwa_gripper_description/urdf/iiwa_gripper.urdf.xacro (robot description, xacro)
@@ -9,5 +9,5 @@
   <xacro:arg name="hardware_interface" default="PositionJointInterface"/>
   <xacro:arg name="robot_name" default="iiwa"/>
-  <xacro:arg name="origin_xyz" default="0.2 0 1.0"/>
+  <xacro:arg name="origin_xyz" default="0.2 0 0.97"/>
   <xacro:arg name="origin_rpy" default="0 0 0"/>
   <!--  Define the origin of your 3D space
@@ -17,9 +17,9 @@
   -->
   <!--     <link name="world"/> -->
-  <link name="world">
+  <link name="suporte">
     <inertial>
-      <origin xyz="0.385 0.5 0.3" rpy="0 0 0"/>
+      <origin xyz="0.385 0 0.3" rpy="0 0 0"/>
       <mass value="100"/>
-      <inertia ixx="11.33"  ixy="0"  ixz="0" iyy="13.27" iyz="0" izz="7.94" />
+      <inertia ixx="11.33"  ixy="0"  ixz="0" iyy="7.94" iyz="0" izz="13.27" />
     </inertial>
     <visual>
@@ -31,16 +31,42 @@
     </visual>
     <collision>
-      <origin xyz="0.40 0 0.499" rpy="-1.57 0 0"/>
+      <origin xyz="0.40 0 0.49" rpy="0 0 0"/>
       <geometry>
-        <box size="0.75 1.0 0.6"/>
+        <box size="0.75 0.6 0.98"/>
 	      <!--mesh filename="package://iiwa_gripper_description/meshes/collision/suporte.stl"/-->
       </geometry>
     </collision>
+    <!-- adding more boxes to improve the collision element -->
+    <collision>
+      <origin xyz="0.285 0.255 1.0" rpy="0 0 0"/>
+      <geometry>
+        <box size="0.285 0.056 0.06"/>
+      </geometry>
+    </collision>
+    <collision>
+      <origin xyz="0.285 -0.257 1.0" rpy="0 0 0"/>
+      <geometry>
+        <box size="0.285 0.056 0.06"/>
+      </geometry>
+    </collision>
+    <collision>
+      <origin xyz="0.595 0 1.01" rpy="0 0 0"/>
+      <geometry>
+        <box size="0.34 0.59 0.09"/>
+      </geometry>
+    </collision>
   </link>
-  <gazebo reference="world">
-    <static>true</static>
+  <link name="link_suporte">
+   </link>
+  <joint name="suporte_joint" type="fixed">
+     <parent link="link_suporte"/>
+     <child link="suporte"/>
+   </joint>
+  <gazebo reference="link_suporte">
+    <!-- <static>true</static> -->
+    <static>false</static>
   </gazebo>
   <!-- Here we insert an iiwa14 robot in the scene, it's origin is just on top of the box previously defined. You can use 0,0,0 if you don't have that. -->
-  <xacro:iiwa14 hardware_interface="$(arg hardware_interface)" robot_name="$(arg robot_name)" parent="world">
+  <xacro:iiwa14 hardware_interface="$(arg hardware_interface)" robot_name="$(arg robot_name)" parent="suporte">
     <origin xyz="$(arg origin_xyz)" rpy="$(arg origin_rpy)" />
   </xacro:iiwa14>

File: iiwa_surgery_description/urdf/iiwa14_surgery.urdf.xacro (robot description, xacro)
@@ -7,5 +7,5 @@
   <xacro:arg name="hardware_interface" default="PositionJointInterface"/>
   <xacro:arg name="robot_name" default="iiwa"/>
-  <xacro:arg name="origin_xyz" default="0 0 0"/>
+  <xacro:arg name="origin_xyz" default="0.2 0 0.97"/>
   <xacro:arg name="origin_rpy" default="0 0 0"/>
   <!-- Fix to world just for testing -->
@@ -25,12 +25,37 @@
     </visual>
     <collision>
-      <origin xyz="0.40 0 0.499" rpy="-1.57 0 0"/>
+      <origin xyz="0.40 0 0.49" rpy="0 0 0"/>
       <geometry>
-        <box size="0.75 1.0 0.6"/>
+        <box size="0.75 0.6 0.98"/>
 	      <!--mesh filename="package://iiwa_gripper_description/meshes/collision/suporte.stl"/-->
       </geometry>
     </collision>
+    <!-- adding more boxes to improve the collision element -->
+    <collision>
+      <origin xyz="0.285 0.255 1.0" rpy="0 0 0"/>
+      <geometry>
+        <box size="0.285 0.056 0.06"/>
+      </geometry>
+    </collision>
+    <collision>
+      <origin xyz="0.285 -0.257 1.0" rpy="0 0 0"/>
+      <geometry>
+        <box size="0.285 0.056 0.06"/>
+      </geometry>
+    </collision>
+    <collision>
+      <origin xyz="0.595 0 1.01" rpy="0 0 0"/>
+      <geometry>
+        <box size="0.34 0.59 0.09"/>
+      </geometry>
+    </collision>
   </link>
-  <gazebo reference="suporte">
+  <link name="link_suporte">
+   </link>
+  <joint name="suporte_joint" type="fixed">
+     <parent link="link_suporte"/>
+     <child link="suporte"/>
+   </joint>
+  <gazebo reference="link_suporte">
     <!-- <static>true</static> -->
     <static>false</static>
