Commit message: spawn_tool.py spawns the tool based on iiwa end effectors position and orientation

File: iiwa_surgery_description/urdf/iiwa14.xacro (robot description, xacro)
@@ -295,5 +295,5 @@
       <parent link="${robot_name}_link_7"/>
       <child link="${robot_name}_link_ee"/>
-      <origin xyz="0 0 0.045" rpy="0 0 0"/>
+      <origin xyz="0 0 0.05" rpy="0 0 0"/>
     </joint>
     <link name="${robot_name}_link_ee">
