Commit message: Added Collada 3D models for the visualization of some objects and the the tools (pen support, drill and tms). The origin of the tools got deslocated after the export for collada, so the rotation, x and y axis are correctd on the SDF model. The z axis is corrected for each tool in the python script spawn_tool.py

File: iiwa_surgery_description/urdf/iiwa14_surgery.urdf.xacro (robot description, xacro)
@@ -18,8 +18,8 @@
     </inertial>
     <visual>
-      <origin xyz="0.4 0 0" rpy="-1.57 0 0"/>
+      <origin xyz="0.4 0 0" rpy="0 0 0"/>
       <geometry>
         <!--box size="0.77 1.0 0.6"/-->
-	      <mesh filename="package://iiwa_surgery_description/meshes/collision/suporte.stl"/>
+	      <mesh filename="package://iiwa_surgery_description/meshes/visual/montagem_modulo.dae"/>
       </geometry>
     </visual>

Commit message: Update minor changes and name changes

File: iiwa_surgery_description/urdf/iiwa14_surgery.urdf.xacro (robot description, xacro)
@@ -9,6 +9,5 @@
   <xacro:arg name="origin_xyz" default="0.2 0 0.97"/>
   <xacro:arg name="origin_rpy" default="0 0 0"/>
-  <!-- Fix to world just for testing -->
-  <!-- <link name="world"/> -->
+  <!-- link over which the robot is attached -->
   <link name="suporte">
     <inertial>
@@ -20,5 +19,4 @@
       <origin xyz="0.4 0 0" rpy="0 0 0"/>
       <geometry>
-        <!--box size="0.77 1.0 0.6"/-->
 	      <mesh filename="package://iiwa_surgery_description/meshes/visual/montagem_modulo.dae"/>
       </geometry>
